File: board-design/pico-gps-datalogger/pico-gps-datalogger.kicad_pcb (KiCad board)
At the start: 2 copper layers, 88.7 x 83.2 mm, 23 parts, among them J1 Conn_01x08_Female, J2 Conn_01x09_Female, J3 Conn_01x02_Female, J4 Conn_01x06_Female, SW1 SW_Push, SW2 SW_Push, SW3 SW_Push, SW4 SW_SPDT, SW5 Power Switch, U1 AMS1117-3.3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

Commit message: updated pcb a bit, to power pico with 5v not 3v3 as it doesn't seem to like that. Added datasheet for GPS.
Connections:
- SW4 pad 1: +3.3V -> VBUS
Routing:
- net +3.3V: track 234.0 -> 179.1 mm
- net VBUS: track 20.1 -> 62.8 mm
- net Net-(SW3-Pad1): vias 4 -> 2
Other:
- board text added: "Mark McGookin Raspberry Pi Pico - SPI Screen - Neopixel - SD Card - GPS Logger Dec 2022 v0.4"
- board text removed: "Mark McGookin Raspberry Pi Pico - SPI Screen - Neopixel - SD Card - GPS Logger Dec 2022 v0.3"
